File: KiCad/beacon_rp2040/beacon_rp2040.kicad_sch (KiCad schematic)
At the start: 17 parts, among them J1 CONNECTIONS, Q1 2N7002, U1 RP2040-ZERO, U3 RS3002-5.0YF5

Commit message: Status LED: red keyed blink during TX, steady green in pause
- WS2812 follows the keying: red while the tone/key sounds, dark in the gaps
- steady green between transmissions (pause and idle)
- removed the old 500 ms blink timer
- firmware/Beacon-v0.1.uf2 rebuilt
Parts:
- removed L2: 10u, Inductor_SMD:L_1206_3216Metric, symbol Device:L
- added D1: MBR0540, Diode_SMD:D_SOD-123, symbol Diode:MBR0540
- added D2: LED_CW, LED_SMD:LED_1206_3216Metric, symbol Device:LED
- added J2: GPIO, symbol Connector_Generic:Conn_01x10
- added J3: GND, symbol Connector_Generic:Conn_01x03
- added J4: 5V, symbol Connector_Generic:Conn_01x03
- added R4: 1k, Resistor_SMD:R_1206_3216Metric, symbol Device:R
Connections:
- net +5V: now also D1.1 (K), J4.1 (Pin_1), J4.2 (Pin_2), J4.3 (Pin_3)
- net GND: now also D2.1 (K), J2.10 (Pin_10), J3.1 (Pin_1), J3.2 (Pin_2), J3.3 (Pin_3)
- net at Q1.1 (G), R3.2, U1.14 (GP13): now also R4.1
- net at U1.1 (GP0): now also J2.1 (Pin_1)
- net at U1.2 (GP1): now also J2.2 (Pin_2)
- net at U1.3 (GP2): now also J2.3 (Pin_3)
- net at U1.4 (GP3): now also J2.4 (Pin_4)
- net at U1.5 (GP4): now also J2.5 (Pin_5)
- net at U1.6 (GP5): now also J2.6 (Pin_6)
- net at U1.7 (GP6): now also J2.7 (Pin_7)
- net at U1.8 (GP7): now also J2.8 (Pin_8)
- net at U1.9 (GP8): now also J2.9 (Pin_9)
- net at C11.1, C12.1, C13.1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: now also D1.2 (A)
- new net: D2.2 (A), R4.2
- no-connect marks 0 -> 9
