File: KiCad/beacon_rp2040/beacon_rp2040.kicad_sch (KiCad schematic)
At the start: 22 parts, among them J1 CONNECTIONS, J2 GPIO, J3 GND, J4 5V, Q1 2N7002, U1 RP2040-ZERO, U3 RS3002-5.0YF5

Commit message: Controller board: schematic, PCB, Gerbers, BOM; README hardware docs
- KiCad schematic and routed 2-layer PCB (75 x 32 mm): LM7805 supply
  with reverse-polarity and USB isolation diodes, audio attenuator with
  low-pass filter, BC817 open-collector PTT/CW outputs, Vin divider on
  GP26, GPIO/5V/GND expansion headers, M3 mounting holes
- Schematic PDF, Gerber + drill files (also zipped), interactive BOM
- Schematic and 3D view images in pics/
- README: board description, J1 pinout, outputs, power, expansion
  headers, manufacturing files and BOM; GUI download is now the zip
- VS Code CMake Tools builds into code/Beacon/build like the scripts

Co-Authored-By: Claude Opus 5.5 <noreply@anthropic.com>
Parts:
- removed C1: 10uF, Capacitor_THT:CP_Radial_D5.0mm_P2.50mm, symbol Device:C_Polarized
- removed D8: LL4148, Diode_SMD:D_MiniMELF, symbol Diode:LL4148
- removed J2: GPIO, symbol Connector_Generic:Conn_01x10
- removed Q1: 2N7002, Package_TO_SOT_SMD:SOT-23, symbol Transistor_FET:2N7002
- removed U3: RS3002-5.0YF5, Package_TO_SOT_SMD:SOT-23-5, symbol Regulator_Linear:AP2112K-3.3
- added C3, C5: 100n, Capacitor_SMD:C_1206_3216Metric, symbol Device:C
- added C4: 10u, Capacitor_SMD:C_1206_3216Metric, symbol Device:C
- added C6: 47n, Capacitor_SMD:C_1206_3216Metric, symbol Device:C
- added D3: LED_PTT, Connector_PinHeader_2.54mm:PinHeader_1x02_P2.54mm_Vertical, symbol Device:LED
- added D4: MBR0540, Diode_SMD:D_SOD-123, symbol Diode:MBR0540
- added H1, H2, H3, H4: MountingHole_Pad, MountingHole:MountingHole_3.2mm_M3_DIN965_Pad, symbol Mechanical:MountingHole_Pad
- added J2: GPIOs, Connector_PinHeader_2.54mm:PinHeader_1x18_P2.54mm_Vertical, symbol Connector_Generic:Conn_01x18
- added Q3, Q4: BC817, Package_TO_SOT_SMD:SOT-23-3, symbol Transistor_BJT:BC817W
- added R10, R6, R9: 1k, Resistor_SMD:R_1206_3216Metric, symbol Device:R
- added R5, R8: 10k, Resistor_SMD:R_1206_3216Metric, symbol Device:R
- added R7: 100k, Resistor_SMD:R_1206_3216Metric, symbol Device:R
- added U2: LM7805_TO220, Package_TO_SOT_THT:TO-220-3_Vertical, symbol Regulator_Linear:LM7805_TO220
- D2: footprint LED_SMD:LED_1206_3216Metric -> Connector_PinHeader_2.54mm:PinHeader_1x02_P2.54mm_Vertical
- J3, J4: footprint (none) -> Connector_PinHeader_2.54mm:PinHeader_1x03_P2.54mm_Vertical
- R1: value 10k -> 34k
Connections:
- net GND: now also C3.1, C5.1, C6.1, D3.1 (K), H1.1, H2.1, H3.1, H4.1, J2.18 (Pin_18), Q3.2 (E), Q4.2 (E), R5.1, R8.2, U2.2 (GND)
- net CW: now reaches R3.2, R4.1
- net CW: now also U1.8 (GP7), R9.2; no longer U1.14 (GP13)
- net at C10.1, C14.1, C9.1: now also D4.1 (K), R7.2, U2.1 (VI)
- net at J1.1 (Pin_1): now also D4.2 (A)
- net at C11.1, C12.1, C13.1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: now also U2.3 (VO)
- net at C2.2, J1.4 (Pin_4): now also Q4.3 (C)
- net GP0: now reaches U1.1 (GP0)
- net GP0: now also J2.2 (Pin_2)
- net GP9: now reaches U1.10 (GP9)
- net GP9: now also J2.10 (Pin_10)
- net GP10: now reaches U1.11 (GP10)
- net GP10: now also J2.11 (Pin_11)
- net GP11: now reaches U1.12 (GP11)
- net GP11: now also J2.12 (Pin_12)
- net GP12: now reaches U1.13 (GP12)
- net GP12: now also J2.13 (Pin_13)
- net PTT: now reaches U1.15 (GP14)
- net PTT: now also R10.2, R5.2, R6.1
- net at U1.17 (GP26): now also C5.2, R7.1, R8.1
- net GP27: now reaches U1.18 (GP27)
- net GP27: now also J2.15 (Pin_15)
- net GP28: now reaches U1.19 (GP28)
- net GP28: now also J2.16 (Pin_16)
- net GP1: now reaches U1.2 (GP1)
- net GP1: now also J2.3 (Pin_3)
- net GP29: now reaches U1.20 (GP29)
- net GP29: now also J2.17 (Pin_17)
- net 3.3V: now reaches U1.21 (3V3)
- net 3.3V: now also J2.1 (Pin_1)
- net GP2: now reaches U1.3 (GP2)
- net GP2: now also J2.4 (Pin_4)
- net GP3: now reaches U1.4 (GP3)
- net GP3: now also J2.5 (Pin_5)
- net GP4: now reaches U1.5 (GP4)
- net GP4: now also J2.6 (Pin_6)
- net GP5: now reaches U1.6 (GP5)
- net GP5: now also J2.7 (Pin_7)
- net GP6: now reaches U1.7 (GP6)
- net GP6: now also J2.8 (Pin_8)
- net GP8: now reaches U1.9 (GP8)
- net GP8: now also J2.9 (Pin_9)
- net at J1.3 (Pin_3): now also C4.2
- net at J1.5 (Pin_5): now also C3.2, Q3.3 (C)
- net at R1.1, R2.1: now also C4.1, C6.2
- new net: Q3.1 (B), R10.1
- new net: D3.2 (A), R6.2
- new net: Q4.1 (B), R9.1
- new net GP13: J2.14 (Pin_14), U1.14 (GP13)
- no-connect marks 9 -> 0
Other:
- title: (none) -> Beacon for any rig
